Commit message: 与实体机械臂同样初始位姿的求解器

File: src/mrx_t4_a00_new/urdf/mrx_t4_a00_new.urdf (robot description, URDF)
Before this commit: robot mrx_t4_a00_new, 7 links, 6 joints
Links:
- link base_link: geometry 
Joints:
- joint armA_to_armB: limit lower=0 upper=2.05948852 effort=300 velocity=1 -> lower=-1.51843645 upper=0.48869219 effort=300 velocity=1; origin xyz=0 -0.113 0.03375 rpy=0 -1.5708 1.5708 -> xyz=0 -0.113 0.03375 rpy=0 -1.5708 0
- joint armB_to_armC: limit lower=-2.5830873 upper=1.5358897418 effort=300 velocity=1 -> lower=-1.01229096 upper=3.10668606 effort=300 velocity=1
- joint armC_to_armD: origin xyz=0 -0.25 0.03 rpy=1.5708 0 0 -> xyz=0.25 0 0.03 rpy=1.5708 0 3.14159
- joint base_to_armA: limit lower=-2.757620 upper=2.757620 effort=300 velocity=1 -> lower=-2.75762022 upper=2.75762022 effort=300 velocity=1

File: src/mrx_t4_a00_new/urdf/mrx_t4_a00_new_backup.urdf (robot description, URDF)
Before this commit: robot mrx_t4_a00_new, 6 links, 5 joints
Links:
- added link vt_hand
- link base_link: mass 500 -> None
Joints:
- added joint armD_to_vthand: type fixed, parent armD, child vt_hand, origin xyz=0 0 0.15 rpy=1.5708 -1.5708 0
- joint armA_to_armB: limit lower=-1.5708 upper=0.349065 effort=300 velocity=1 -> lower=0 upper=2.05948852 effort=300 velocity=1; origin xyz=0 -0.113 0.03375 rpy=0 -1.5708 0 -> xyz=0 -0.113 0.03375 rpy=0 -1.5708 1.5708
- joint armB_to_armC: limit lower=-2.0944 upper=2.0944 effort=300 velocity=1 -> lower=-2.5830873 upper=1.5358897418 effort=300 velocity=1
- joint armC_to_armD: origin xyz=0.25 0 0.03 rpy=1.5708 0 3.1416 -> xyz=0 -0.25 0.03 rpy=1.5708 0 0
- joint base_to_armA: limit lower=-2.967 upper=2.967 effort=300 velocity=1 -> lower=-2.757620 upper=2.757620 effort=300 velocity=1
