Commit message: backup on 11/8/2018

File: src/mrx_t4_a00_new/urdf/kinect.xacro (robot description, xacro)
@@ -17,5 +17,5 @@
         </link>
         <joint name="${prefix}_optical_joint" type="fixed">
-            <origin xyz="0 0 0" rpy="0 0 0" />
+            <origin xyz="0 0 0" rpy="-1.5708 0 -1.5708" />
             <parent link="${prefix}_link"/>
             <child link="${prefix}_frame_optical"/>
@@ -26,5 +26,5 @@
             <sensor type="depth" name="${prefix}">
                 <always_on>true</always_on>
-                <update_rate>20.0</update_rate>
+                <update_rate>1</update_rate>
                 <camera>
                     <horizontal_fov>${60.0*M_PI/180}</horizontal_fov>

File: src/mrx_t4_a00_new/urdf/mrx_t4_a00_new_with_kinect_gazebo.xacro (robot description, xacro)
@@ -6,4 +6,10 @@
   <xacro:property name="kinect_offset_z" value="1.2"/>
   <xacro:property name="M_PI" value="3.141592654"/>
+  <!-- fixed frame in gazebo -->
+  <link name="world" />
+  <joint name="world_base_link_joint" type="fixed">
+      <parent link="world" />
+      <child link="base_link"/>
+  </joint>
   <link name="base_link">
     <!--
